Commit message: Combine objs

File: src/assets/furniture/urdf/obstacle.urdf (robot description, URDF)
Before this commit: robot obstacle, 4 links, 3 joints
Links:
- removed link obstacle_front
- removed link obstacle_left
- removed link obstacle_right
- link base_link: geometry collision mesh filename=../mesh/obstacle.obj; visual mesh filename=../mesh/obstacle.obj
Joints:
- removed joint base_to_front
- removed joint front_to_left
- removed joint front_to_right
