Commit message: changes for saving residual actions + base actions + visualizing them in isaac sim

File: src/assets/furniture/urdf/square_table/square_table_leg4.urdf (robot description, URDF)
Before this commit: robot square_table_leg4, 1 links, 0 joints
Links:
- link square_table_leg4: geometry collision mesh filename=../mesh/square_table/square_table_leg4.obj scale=1 1 1
